Commit message: 20230719

File: robot_liuzu/urdf/robot_liuzu.urdf (robot description, URDF)
Before this commit: robot robot_liuzu, 20 links, 19 joints
Joints:
- joint thigh_rb: limit lower=-0.2 upper=0.4 effort=100 velocity=1.570796 -> lower=-0.4 upper=0.2 effort=100 velocity=1.570796
- joint thigh_rm: limit lower=-0.2 upper=0.4 effort=100 velocity=1.570796 -> lower=-0.4 upper=0.2 effort=100 velocity=1.570796

Commit message: 20230720

File: robot_liuzu/urdf/robot_liuzu.urdf (robot description, URDF)
Before this commit: robot robot_liuzu, 20 links, 19 joints
Joints:
- joint body_lb: limit lower=-0.471 upper=0.471 effort=100 velocity=1.570796 -> lower=-0.471 upper=0.471 effort=200 velocity=1.570796
- joint body_lf: limit lower=-0.471 upper=0.471 effort=100 velocity=1.570796 -> lower=-0.471 upper=0.471 effort=200 velocity=1.570796
- joint body_lm: limit lower=-0.471 upper=0.471 effort=100 velocity=1.570796 -> lower=-0.471 upper=0.471 effort=200 velocity=1.570796
- joint body_rb: limit lower=-0.471 upper=0.471 effort=100 velocity=1.570796 -> lower=-0.471 upper=0.471 effort=200 velocity=1.570796
- joint body_rf: limit lower=-0.471 upper=0.471 effort=100 velocity=1.570796 -> lower=-0.471 upper=0.471 effort=200 velocity=1.570796
- joint body_rm: limit lower=-0.471 upper=0.471 effort=100 velocity=1.570796 -> lower=-0.471 upper=0.471 effort=200 velocity=1.570796
- joint shank_lb: limit lower=-0.6 upper=0.1 effort=100 velocity=1.570796 -> lower=-0.3 upper=0.1 effort=200 velocity=1.570796
- joint shank_lf: limit lower=-0.6 upper=0.1 effort=100 velocity=1.570796 -> lower=-0.3 upper=0.1 effort=200 velocity=1.570796
- joint shank_lm: limit lower=-0.6 upper=0.1 effort=100 velocity=1.570796 -> lower=-0.3 upper=0.1 effort=200 velocity=1.570796
- joint shank_rb: limit lower=-0.1 upper=0.6 effort=100 velocity=1.570796 -> lower=-0.1 upper=0.3 effort=200 velocity=1.570796
- joint shank_rf: limit lower=-0.1 upper=0.6 effort=100 velocity=1.570796 -> lower=-0.1 upper=0.3 effort=200 velocity=1.570796
- joint shank_rm: limit lower=-0.1 upper=0.6 effort=100 velocity=1.570796 -> lower=-0.1 upper=0.3 effort=200 velocity=1.570796
- joint thigh_lb: limit lower=-0.2 upper=0.4 effort=100 velocity=1.570796 -> lower=-0.2 upper=0.4 effort=200 velocity=1.570796
- joint thigh_lf: limit lower=-0.2 upper=0.4 effort=100 velocity=1.570796 -> lower=-0.2 upper=0.4 effort=200 velocity=1.570796
- joint thigh_lm: limit lower=-0.2 upper=0.4 effort=100 velocity=1.570796 -> lower=-0.2 upper=0.4 effort=200 velocity=1.570796
- joint thigh_rb: limit lower=-0.4 upper=0.2 effort=100 velocity=1.570796 -> lower=-0.4 upper=0.2 effort=200 velocity=1.570796
- joint thigh_rf: limit lower=-0.4 upper=0.2 effort=100 velocity=1.570796 -> lower=-0.4 upper=0.2 effort=200 velocity=1.570796
- joint thigh_rm: limit lower=-0.4 upper=0.2 effort=100 velocity=1.570796 -> lower=-0.4 upper=0.2 effort=200 velocity=1.570796
